Commit message: Modify : GNSSトピック名変更
ubloxのGNSSのトピック名が変更となったため
関連するパッケージのトピック名を再検討し変更

xacroからsdfへの変換にてエラーとなったため
realsense_linkのbox sizeの指定を修正

File: rccar_description/models/rccar/rccar.gazebo.urdf.xacro (robot description, xacro)
@@ -30,5 +30,5 @@
         <frame_name>gps_link</frame_name>
         <ros>
-          <remapping>~/out:=/fix</remapping>
+          <remapping>~/out:=/gnss/fix</remapping>
         </ros>
       </plugin>
@@ -53,7 +53,5 @@
       <origin xyz="0.0 0.0 0.0" rpy="-1.57 0 -1.57" />
       <geometry>
-        <box>
-          <size>0.02505 0.09 0.025</size>
-        </box>
+        <box size="0.02505 0.09 0.025" />
       </geometry>
       <!--
@@ -66,7 +64,5 @@
       <origin xyz="0.0 0.0 0.0" rpy="-1.57 0 -1.57" />
       <geometry>
-        <box>
-          <size>0.02505 0.09 0.025</size>
-        </box>
+        <box size="0.02505 0.09 0.025" />
       </geometry>
       <!--

File: rccar_description/models/rccar/rccar.urdf (robot description, URDF)
Before this commit: robot rccar, 25 links, 24 joints
Links:
- link realsense_link: geometry collision box size=0.02505 0.09 0.025; visual box size=0.02505 0.09 0.025

Commit message: Modify : 重複link削除
camera_linkと重複しているrealsense_linkを削除

File: rccar_description/models/rccar/rccar.gazebo.urdf.xacro (robot description, xacro)
@@ -49,39 +49,5 @@
     </sensor>
   </gazebo>
-  <link name="realsense_link">
-    <visual>
-      <origin xyz="0.0 0.0 0.0" rpy="-1.57 0 -1.57" />
-      <geometry>
-        <box size="0.02505 0.09 0.025" />
-      </geometry>
-      <!--
-      <geometry>
-        <mesh filename="file://$(find realsense2_description)/meshes/d435.dae" />
-      </geometry>
-      -->
-    </visual>
-    <collision>
-      <origin xyz="0.0 0.0 0.0" rpy="-1.57 0 -1.57" />
-      <geometry>
-        <box size="0.02505 0.09 0.025" />
-      </geometry>
-      <!--
-      <geometry>
-        <mesh filename="file://$(find realsense2_description)/meshes/d435.dae" />
-      </geometry>
-      -->
-    </collision>
-    <inertial>
-      <mass value="0.564" />
-      <inertia ixx="0.001" ixy="0.000" ixz="0.000" iyy="0.001" iyz="0.000" izz="0.001" />
-    </inertial>
-  </link>
-  <joint name="realsense_joint" type="fixed">
-    <parent link="camera_link" />
-    <child link="realsense_link" />
-    <axis xyz="0 0 0" rpy="0 0 0" />
-    <origin xyz="0 0 0" rpy="0 0 0" />
-  </joint>
-  <gazebo reference="realsense_link">
+  <gazebo reference="camera_link">
     <sensor name="cameradepth" type="depth">
       <camera name="camera">

File: rccar_description/models/rccar/rccar.urdf (robot description, URDF)
Before this commit: robot rccar, 25 links, 24 joints
Links:
- removed link realsense_link
Joints:
- removed joint realsense_joint
