Commit message: Modify : LiDAR-Odometry追加
LiDARのOdometryを追加

File: rccar_description/models/rccar-bronco/rccar-bronco.gazebo.urdf.xacro (robot description, xacro)
@@ -212,5 +212,5 @@
     <sensor name="lidar_imu" type="imu">
       <always_on>true</always_on>
-      <update_rate>200</update_rate>
+      <update_rate>10</update_rate>
       <plugin filename="libgazebo_ros_imu_sensor.so" name="lidar_imu_plugin">
         <frame_name>lidar_link</frame_name>

File: rccar_description/models/rccar-bronco/rccar-bronco.urdf.xacro (robot description, xacro)
@@ -38,5 +38,5 @@
       <geometry>
         <box size="0.055 0.060 0.0225" />
-      </geometry>livox_laser_simulation_ros2
+      </geometry>
       <material name="black"/>
     </visual>

Commit message: Modify : LiDAR-Localization追加
LiDARの3D(PointCloud)でのLocalizationを追加

File: rccar_description/models/rccar-bronco/rccar-bronco.gazebo.urdf.xacro (robot description, xacro)
@@ -212,5 +212,5 @@
     <sensor name="lidar_imu" type="imu">
       <always_on>true</always_on>
-      <update_rate>10</update_rate>
+      <update_rate>200</update_rate>
       <plugin filename="libgazebo_ros_imu_sensor.so" name="lidar_imu_plugin">
         <frame_name>lidar_link</frame_name>
@@ -221,3 +221,7 @@
     </sensor>
   </gazebo>
+  <!-- <xacro:include filename="$(find rccar_description)/urdf/VLP-16.urdf.xacro" />
+  <xacro:VLP-16 parent="lidar_link" name="velodyne" topic="/velodyne_points" organize_cloud="false" hz="10" samples="440" gpu="false">
+    <origin xyz="0 0 0" rpy="0 0 0" />
+  </xacro:VLP-16> -->
 </robot>

Commit message: Modify : BRONCOモデル変更
LiDARのLinkのlivox_frameを追加
pointcloud_to_laserscanのパラメータをコンフィグファイルとして外出し

File: rccar_description/models/rccar-bronco/rccar-bronco.gazebo.urdf.xacro (robot description, xacro)
@@ -208,5 +208,5 @@
     </plugin>
   </gazebo>
-  <gazebo reference="lidar_link">
+  <gazebo reference="livox_frame">
     <gravity>true</gravity>
     <sensor name="lidar_imu" type="imu">
@@ -214,5 +214,5 @@
       <update_rate>200</update_rate>
       <plugin filename="libgazebo_ros_imu_sensor.so" name="lidar_imu_plugin">
-        <frame_name>lidar_link</frame_name>
+        <frame_name>livox_frame</frame_name>
         <ros>
           <remapping>~/out:=/lidar/imu_raw</remapping>

File: rccar_description/models/rccar-bronco/rccar-bronco.urdf (robot description, URDF)
Before this commit: robot rccar_bronco, 25 links, 24 joints
Links:
- added link livox_frame, mass 0.1; visual box size=0.1 0.06 0.06
- link lidar_link: mass 0.1 -> None; geometry 
Joints:
- removed joint lidar_link_joint
- added joint base_link_to_lidar_link: type fixed, parent base_link, child lidar_link, origin xyz=-0.094 0.0 0.309 rpy=0 0 0
- added joint livox_frame_joint: type fixed, parent lidar_link, child livox_frame, origin xyz=0 0 0 rpy=0 0 0

File: rccar_description/models/rccar-bronco/rccar-bronco.urdf.xacro (robot description, xacro)
@@ -50,6 +50,12 @@
     <origin xyz="-0.0239 0.0 0.279" rpy="0 0 0"/>
   </xacro:sensor_d435i>
-  <xacro:mid360 name="lidar_link" parent="base_link" topic="lidar/points_raw">
+  <link name="lidar_link"/>
+  <joint name="base_link_to_lidar_link" type="fixed">
+    <parent link="base_link"/>
+    <child link="lidar_link" />
     <origin xyz="-0.094 0.0 0.309" rpy="0 0 0"/>
+  </joint>
+  <xacro:mid360 name="livox_frame" parent="lidar_link" topic="lidar/points_raw">
+    <origin xyz="0 0 0" rpy="0 0 0"/>
   </xacro:mid360>
   <xacro:macro name="wheel" params="prefix suffix x y z mode">

Commit message: Modify : BRONCO/UNIMOGモデル変更
カメラのIMUのLinkをcamera_imu_optical_frameに変更

File: rccar_description/models/rccar-bronco/rccar-bronco.gazebo.urdf.xacro (robot description, xacro)
@@ -35,6 +35,6 @@
     </sensor>
   </gazebo>
-  <!--<gazebo reference="camera_imu_optical_frame">-->
-  <gazebo reference="camera_gyro_optical_frame">
+  <gazebo reference="camera_imu_optical_frame">
+  <!-- <gazebo reference="camera_gyro_optical_frame"> -->
     <gravity>true</gravity>
     <sensor name="camera_imu" type="imu">
@@ -42,5 +42,6 @@
       <update_rate>200</update_rate>
       <plugin filename="libgazebo_ros_imu_sensor.so" name="camera_imu_plugin">
-        <frame_name>camera_gyro_optical_frame</frame_name>
+        <frame_name>camera_imu_optical_frame</frame_name>
+        <!-- <frame_name>camera_gyro_optical_frame</frame_name> -->
         <ros>
           <remapping>~/out:=/camera/imu_raw</remapping>

File: rccar_description/models/rccar-bronco/rccar-bronco.urdf (robot description, URDF)
Before this commit: robot rccar_bronco, 26 links, 25 joints
Links:
- added link camera_imu_optical_frame
Joints:
- added joint gyro_optical_to_imu_optical: type fixed, parent camera_gyro_optical_frame, child camera_imu_optical_frame, origin xyz=0 0 0 rpy=0 0 0

File: rccar_description/models/rccar-bronco/rccar-bronco.urdf.xacro (robot description, xacro)
@@ -50,4 +50,10 @@
     <origin xyz="-0.0239 0.0 0.279" rpy="0 0 0"/>
   </xacro:sensor_d435i>
+  <link name="camera_imu_optical_frame"/>
+  <joint name="gyro_optical_to_imu_optical" type="fixed">
+    <parent link="camera_gyro_optical_frame"/>
+    <child link="camera_imu_optical_frame" />
+    <origin xyz="0 0 0" rpy="0 0 0"/>
+  </joint>
   <link name="lidar_link"/>
   <joint name="base_link_to_lidar_link" type="fixed">

File: rccar_description/models/rccar-unimog/rccar-unimog.gazebo.urdf.xacro (robot description, xacro)
@@ -35,6 +35,6 @@
     </sensor>
   </gazebo>
-  <!--<gazebo reference="camera_imu_optical_frame">-->
-  <gazebo reference="camera_gyro_optical_frame">
+  <gazebo reference="camera_imu_optical_frame">
+  <!-- <gazebo reference="camera_gyro_optical_frame"> -->
     <gravity>true</gravity>
     <sensor name="camera_imu" type="imu">
@@ -42,5 +42,6 @@
       <update_rate>200</update_rate>
       <plugin filename="libgazebo_ros_imu_sensor.so" name="imu_plugin">
-        <frame_name>camera_gyro_optical_frame</frame_name>
+        <frame_name>camera_imu_optical_frame</frame_name>
+        <!-- <frame_name>camera_gyro_optical_frame</frame_name> -->
         <ros>
           <remapping>~/out:=/camera/imu_raw</remapping>

File: rccar_description/models/rccar-unimog/rccar-unimog.urdf (robot description, URDF)
Before this commit: robot rccar-unimog, 24 links, 23 joints
Links:
- added link camera_imu_optical_frame
Joints:
- added joint gyro_optical_to_imu_optical: type fixed, parent camera_gyro_optical_frame, child camera_imu_optical_frame, origin xyz=0 0 0 rpy=0 0 0

File: rccar_description/models/rccar-unimog/rccar-unimog.urdf.xacro (robot description, xacro)
@@ -65,4 +65,10 @@
     <origin xyz="0.09615 0.0 0.185" rpy="0 0 0"/>
   </xacro:sensor_d435i>
+  <link name="camera_imu_optical_frame"/>
+  <joint name="gyro_optical_to_imu_optical" type="fixed">
+    <parent link="camera_gyro_optical_frame"/>
+    <child link="camera_imu_optical_frame" />
+    <origin xyz="0 0 0" rpy="0 0 0"/>
+  </joint>
   <xacro:macro name="wheel" params="prefix suffix x y z mode">
     <link name="${prefix}_${suffix}_mount">

Commit message: Modify : IMU(BNO055)追加
CameraのIMUがLiDARの回転(振動)に影響してしまっているため
LiDARに影響しない位置にBNO055のIMUを追加

File: rccar_description/models/rccar-bronco/rccar-bronco.gazebo.urdf.xacro (robot description, xacro)
@@ -226,3 +226,16 @@
     <origin xyz="0 0 0" rpy="0 0 0" />
   </xacro:VLP-16> -->
+  <gazebo reference="imu_link">
+    <gravity>true</gravity>
+    <sensor name="bno055_imu" type="imu">
+      <always_on>true</always_on>
+      <update_rate>100</update_rate>
+      <plugin filename="libgazebo_ros_imu_sensor.so" name="bno055_imu_plugin">
+        <frame_name>imu_link</frame_name>
+        <ros>
+          <remapping>~/out:=/bno055/imu_raw</remapping>
+        </ros>
+      </plugin>
+    </sensor>
+  </gazebo>
 </robot>

File: rccar_description/models/rccar-bronco/rccar-bronco.urdf (robot description, URDF)
Before this commit: robot rccar_bronco, 27 links, 26 joints
Links:
- added link imu_link
Joints:
- added joint base_link_to_imu_link: type fixed, parent base_link, child imu_link, origin xyz=-0.15 0.0 0.17 rpy=0 0 0

File: rccar_description/models/rccar-bronco/rccar-bronco.urdf.xacro (robot description, xacro)
@@ -65,4 +65,10 @@
     <origin xyz="0 0 0" rpy="0 0 0"/>
   </xacro:mid360>
+  <link name="imu_link"/>
+  <joint name="base_link_to_imu_link" type="fixed">
+    <parent link="base_link"/>
+    <child link="imu_link" />
+    <origin xyz="-0.15 0.0 0.17" rpy="0 0 0"/>
+  </joint>
   <xacro:macro name="wheel" params="prefix suffix x y z mode">
     <link name="${prefix}_${suffix}_mount">
